Commit message: added gps plugin to spot model

File: spot_description/urdf/spot.urdf (robot description, URDF)
Before this commit: robot spot, 27 links, 26 joints
Links:
- added link gps_link, mass 1; collision cylinder length=0.02 radius=0.02; visual cylinder length=0.02 radius=0.02
- link body: mass 32.0 -> 16.0
- link front_left_hip: mass 4.0 -> 2.0
- link front_left_lower_leg: mass 1.0 -> 0.5
- link front_left_upper_leg: mass 2.0 -> 1.0
- link front_right_hip: mass 4.0 -> 2.0
- link front_right_lower_leg: mass 1.0 -> 0.5
- link front_right_upper_leg: mass 2.0 -> 1.0
- link rear_left_hip: mass 4.0 -> 2.0
- link rear_left_lower_leg: mass 1.0 -> 0.5
- link rear_left_upper_leg: mass 2.0 -> 1.0
- link rear_right_hip: mass 4.0 -> 2.0
- link rear_right_lower_leg: mass 1.0 -> 0.5
- link rear_right_upper_leg: mass 2.0 -> 1.0
Joints:
- added joint gps_joint: type fixed, parent base_link, child gps_link
